Commit message: Added separate control for each wheel

File: src/platform_bot/description/robot_platform.xacro (robot description, xacro)
@@ -20,5 +20,5 @@
         </visual>
         <collision>
-            <origin xyz="0.0 0.0 0.5"/>
+            <origin xyz="0.0 0.0 0.05"/>
             <geometry>
                 <box size="0.3 0.2 0.1"/>

File: src/platform_bot/description/ros2_control.xacro (robot description, xacro)
@@ -40,5 +40,5 @@
     <gazebo>
         <plugin filename="libgazebo_ros2_control.so" name="gazebo_ros2_control">
-            <parameters>$(find platform_bot)/config/diff_drive_controller.yaml</parameters>
+            <parameters>$(find platform_bot)/config/mecanum_controler.yaml</parameters>
         </plugin>
     </gazebo>

Commit message: Added wheel macro

File: src/platform_bot/description/robot_platform.xacro (robot description, xacro)
@@ -1,6 +1,12 @@
 <?xml version="1.0"?>
 <robot xmlns:xacro="http://www.ros.org/wiki/xacro">
-    <xacro:include filename="colors.xacro"/>
     <xacro:include filename="inertial.xacro"/>
+    <xacro:include filename="mecanum_wheel.xacro"/>
+    <xacro:property name="body_size_x" value="0.2"/>
+    <xacro:property name="body_size_y" value="0.3"/>
+    <xacro:property name="body_size_z" value="0.1"/>
+    <xacro:property name="wheel_offset_x" value="0.125"/>
+    <xacro:property name="wheel_offset_y" value="0.12"/>
+    <xacro:property name="wheel_offset_z" value="0"/>
     <link name="base_link">
     </link>
@@ -11,19 +17,22 @@
     </joint>
     <!-- Chassis Link -->
+    <material name="chassis_color">
+        <color rgba="1.0 1.0 1.0 1.0"/>
+    </material>
     <link name="chassis_link">
         <visual>
             <origin xyz="0.0 0.0 0.05"/>
             <geometry>
-                <box size="0.3 0.2 0.1"/>
+                <box size="${body_size_x} ${body_size_y} ${body_size_z}"/>
             </geometry>
-            <material name="white"/>
+            <material name="chassis_color"/>
         </visual>
         <collision>
             <origin xyz="0.0 0.0 0.05"/>
             <geometry>
-                <box size="0.3 0.2 0.1"/>
+                <box size="${body_size_x} ${body_size_y} ${body_size_z}"/>
             </geometry>
         </collision>
-        <xacro:inertial_box mass="0.5" x="0.3" y="0.3" z="0.15">
+        <xacro:inertial_box mass="0.5" x="${body_size_x}" y="${body_size_y}" z="${body_size_z}">
             <origin xyz="0.15 0 0.075" rpy="0 0 0"/>
         </xacro:inertial_box>
@@ -33,6 +42,19 @@
     </gazebo>
     <!-- Wheels -->
-    <!-- FL -->
-    <joint name="wheel_fl_joint" type="continuous">
+    <!-- <xacro:macro name="wheels"> -->
+        <xacro:mecanum_wheel prefix="fl" parent="chassis_link">
+            <origin xyz="-${wheel_offset_x} ${wheel_offset_y} ${wheel_offset_z}" rpy="0.0 -${pi/2} 0.0"/>
+        </xacro:mecanum_wheel>
+        <xacro:mecanum_wheel prefix="fr" parent="chassis_link">
+            <origin xyz="${wheel_offset_x} ${wheel_offset_y} ${wheel_offset_z}" rpy="0.0 -${pi/2} 0.0"/>
+        </xacro:mecanum_wheel>
+        <xacro:mecanum_wheel prefix="rl" parent="chassis_link">
+            <origin xyz="-${wheel_offset_x} -${wheel_offset_y} ${wheel_offset_z}" rpy="0.0 -${pi/2} 0.0"/>
+        </xacro:mecanum_wheel>
+        <xacro:mecanum_wheel prefix="rr" parent="chassis_link">
+            <origin xyz="${wheel_offset_x} -${wheel_offset_y} ${wheel_offset_z}" rpy="0.0 -${pi/2} 0.0"/>
+        </xacro:mecanum_wheel>
+    <!-- </xacro:macro> -->
+    <!-- <joint name="wheel_fl_joint" type="continuous">
         <parent link="chassis_link"/>
         <child link="wheel_fl_link"/>
@@ -59,5 +81,4 @@
         <material>Gazebo/Blue</material>
     </gazebo>
-    <!-- FR -->
     <joint name="wheel_fr_joint" type="continuous">
         <parent link="chassis_link"/>
@@ -85,5 +106,4 @@
         <material>Gazebo/Blue</material>
     </gazebo>
-    <!-- RL -->
     <joint name="wheel_rl_joint" type="continuous">
         <parent link="chassis_link"/>
@@ -111,5 +131,4 @@
         <material>Gazebo/Blue</material>
     </gazebo>
-    <!-- RR -->
     <joint name="wheel_rr_joint" type="continuous">
         <parent link="chassis_link"/>
@@ -136,4 +155,4 @@
     <gazebo reference="wheel_rr_link">
         <material>Gazebo/Blue</material>
-    </gazebo>
+    </gazebo> -->
 </robot>

File: src/platform_bot/description/ros2_control.xacro (robot description, xacro)
@@ -5,5 +5,5 @@
             <plugin>gazebo_ros2_control/GazeboSystem</plugin>
         </hardware>
-        <joint name="wheel_fl_joint">
+        <joint name="fl_wheel_joint">
             <command_interface name="velocity">
                 <param name="min">-10</param>
@@ -13,5 +13,5 @@
             <state_interface name="velocity" />
         </joint>
-        <joint name="wheel_fr_joint">
+        <joint name="fr_wheel_joint">
             <command_interface name="velocity">
                 <param name="min">-10</param>
@@ -21,5 +21,5 @@
             <state_interface name="position" />
         </joint>
-        <joint name="wheel_rl_joint">
+        <joint name="rl_wheel_joint">
             <command_interface name="velocity">
                 <param name="min">-10</param>
@@ -29,5 +29,5 @@
             <state_interface name="position" />
         </joint>
-        <joint name="wheel_rr_joint">
+        <joint name="rr_wheel_joint">
             <command_interface name="velocity">
                 <param name="min">-10</param>
