Commit message: Added simple procedural rollers

File: src/platform_bot/description/mecanum_wheel.xacro (robot description, xacro)
@@ -5,4 +5,37 @@
         <color rgba="1 0.3 0.1 1"/>
     </material>
+    <material name="roller_color">
+        <color rgba="0.8 0.6 0.2 1"/>
+    </material>
+    <xacro:macro name="rollers_loop" params="iterator qty prefix parent radius">
+        <joint name="roller_${prefix}_wheel_joint_${iterator}" type="continuous">
+            <origin xyz="${sin((iterator/qty) * 2 * pi) * radius} ${cos((iterator/qty) * 2 * pi) * radius} 0.0" rpy="0.0 0.0 0.0"/>
+            <parent link="${parent}"/>
+            <child link="roller_${prefix}_wheel_link_${iterator}"/>
+            <axis xyz="0 0 1"/>
+        </joint>
+        <link name="roller_${prefix}_wheel_link_${iterator}">
+            <visual>
+                <geometry>
+                    <cylinder radius="0.005" length="0.04"/>
+                </geometry>
+                <material name="roller_color"/>
+            </visual>
+            <collision>
+                <geometry>
+                    <cylinder radius="0.005" length="0.04"/>
+                </geometry>
+            </collision>
+            <xacro:inertial_cylinder mass="0.01" length="0.04" radius="0.0025">
+                <origin xyz="0 0 0" rpy="0 0 0"/>
+            </xacro:inertial_cylinder>
+        </link>
+        <xacro:if value="${iterator}">
+            <xacro:rollers_loop iterator="${iterator-1}" qty="${qty}" prefix="${prefix}" parent="${parent}" radius="${radius}"/>
+        </xacro:if>
+    </xacro:macro>
+    <xacro:macro name="rollers" params="qty prefix parent radius">
+        <xacro:rollers_loop iterator="${qty-1}" qty="${qty}" prefix="${prefix}" parent="${parent}" radius="${radius}"/>
+    </xacro:macro>
     <xacro:macro name="mecanum_wheel" params="prefix parent *origin">
         <joint name="${prefix}_wheel_joint" type="continuous">
@@ -31,4 +64,5 @@
             <material>Gazebo/Blue</material>
         </gazebo>
+        <xacro:rollers qty="5" prefix="${prefix}" parent="${prefix}_wheel_link" radius="0.05"/>
     </xacro:macro>
 </robot>

Commit message: Added Gazebo color reference

File: src/platform_bot/description/mecanum_wheel.xacro (robot description, xacro)
@@ -31,4 +31,7 @@
             </xacro:inertial_cylinder>
         </link>
+        <gazebo reference="roller_${prefix}_wheel_link_${iterator}">
+            <material>Gazebo/Orange</material>
+        </gazebo>
         <xacro:if value="${iterator}">
             <xacro:rollers_loop iterator="${iterator-1}" qty="${qty}" prefix="${prefix}" parent="${parent}" radius="${radius}"/>
@@ -64,5 +67,5 @@
             <material>Gazebo/Blue</material>
         </gazebo>
-        <xacro:rollers qty="5" prefix="${prefix}" parent="${prefix}_wheel_link" radius="0.05"/>
+        <xacro:rollers qty="10" prefix="${prefix}" parent="${prefix}_wheel_link" radius="0.05"/>
     </xacro:macro>
 </robot>

Commit message: Added tilt to rollers

File: src/platform_bot/description/mecanum_wheel.xacro (robot description, xacro)
@@ -8,7 +8,7 @@
         <color rgba="0.8 0.6 0.2 1"/>
     </material>
-    <xacro:macro name="rollers_loop" params="iterator qty prefix parent radius">
+    <xacro:macro name="rollers_loop" params="iterator qty prefix parent radius direction">
         <joint name="roller_${prefix}_wheel_joint_${iterator}" type="continuous">
-            <origin xyz="${sin((iterator/qty) * 2 * pi) * radius} ${cos((iterator/qty) * 2 * pi) * radius} 0.0" rpy="0.0 0.0 0.0"/>
+            <origin xyz="${sin((iterator/qty) * 2 * pi) * radius} ${cos((iterator/qty) * 2 * pi) * radius} 0.0" rpy="${sin((iterator/qty) * 2 * pi) * pi/4 * direction} ${cos((iterator/qty) * 2 * pi) * pi/4 * direction} 0.0"/>
             <parent link="${parent}"/>
             <child link="roller_${prefix}_wheel_link_${iterator}"/>
@@ -35,11 +35,11 @@
         </gazebo>
         <xacro:if value="${iterator}">
-            <xacro:rollers_loop iterator="${iterator-1}" qty="${qty}" prefix="${prefix}" parent="${parent}" radius="${radius}"/>
+            <xacro:rollers_loop iterator="${iterator-1}" qty="${qty}" prefix="${prefix}" parent="${parent}" radius="${radius}" direction="${direction}"/>
         </xacro:if>
     </xacro:macro>
-    <xacro:macro name="rollers" params="qty prefix parent radius">
-        <xacro:rollers_loop iterator="${qty-1}" qty="${qty}" prefix="${prefix}" parent="${parent}" radius="${radius}"/>
+    <xacro:macro name="rollers" params="qty prefix parent radius direction">
+        <xacro:rollers_loop iterator="${qty-1}" qty="${qty}" prefix="${prefix}" parent="${parent}" radius="${radius}" direction="${direction}"/>
     </xacro:macro>
-    <xacro:macro name="mecanum_wheel" params="prefix parent *origin">
+    <xacro:macro name="mecanum_wheel" params="prefix parent *origin direction">
         <joint name="${prefix}_wheel_joint" type="continuous">
             <parent link="${parent}"/>
@@ -67,5 +67,5 @@
             <material>Gazebo/Blue</material>
         </gazebo>
-        <xacro:rollers qty="10" prefix="${prefix}" parent="${prefix}_wheel_link" radius="0.05"/>
+        <xacro:rollers qty="16" prefix="${prefix}" parent="${prefix}_wheel_link" radius="0.05" direction="${direction}"/>
     </xacro:macro>
 </robot>

File: src/platform_bot/description/robot_platform.xacro (robot description, xacro)
@@ -43,14 +43,14 @@
     <!-- Wheels -->
     <!-- <xacro:macro name="wheels"> -->
-        <xacro:mecanum_wheel prefix="fl" parent="chassis_link">
+        <xacro:mecanum_wheel prefix="fl" parent="chassis_link" direction="-1">
             <origin xyz="-${wheel_offset_x} ${wheel_offset_y} ${wheel_offset_z}" rpy="0.0 -${pi/2} 0.0"/>
         </xacro:mecanum_wheel>
-        <xacro:mecanum_wheel prefix="fr" parent="chassis_link">
+        <xacro:mecanum_wheel prefix="fr" parent="chassis_link" direction="1">
             <origin xyz="${wheel_offset_x} ${wheel_offset_y} ${wheel_offset_z}" rpy="0.0 -${pi/2} 0.0"/>
         </xacro:mecanum_wheel>
-        <xacro:mecanum_wheel prefix="rl" parent="chassis_link">
+        <xacro:mecanum_wheel prefix="rl" parent="chassis_link" direction="1">
             <origin xyz="-${wheel_offset_x} -${wheel_offset_y} ${wheel_offset_z}" rpy="0.0 -${pi/2} 0.0"/>
         </xacro:mecanum_wheel>
-        <xacro:mecanum_wheel prefix="rr" parent="chassis_link">
+        <xacro:mecanum_wheel prefix="rr" parent="chassis_link" direction="-1">
             <origin xyz="${wheel_offset_x} -${wheel_offset_y} ${wheel_offset_z}" rpy="0.0 -${pi/2} 0.0"/>
         </xacro:mecanum_wheel>
